Commit message: Set head/neck collisions

File: urdf/jimmy2.urdf.xacro (robot description, xacro)
@@ -3,5 +3,5 @@
     <xacro:property name="mass" value="0.2" />
     <xacro:property name="bracket_mass" value="0.01" />
-    <xacro:property name="ax12_width" value="0.26" />
+    <xacro:property name="ax12_width" value="0.27" />
     <xacro:property name="ax12_height" value="0.5" />
     <xacro:property name="ax12_depth" value="0.4" />
@@ -12,4 +12,6 @@
     <xacro:property name="height3" value="1" /> <!-- Link 3 -->
     <xacro:property name="base_height" value="1.0" />
+    <xacro:property name="package_name" value="test_description" />
+    <xacro:property name="mesh_dir" value="meshes2" />
     <xacro:property name="torso_origin">
         <origin xyz="0 0 ${base_height/2}" rpy="0 0 0"/>
@@ -30,4 +32,7 @@
         <box size="${ax12_width} ${ax12_depth} ${ax12_height}"/>
     </xacro:property>
+    <xacro:property name="ax12_block_collision">
+        <box size="${ax12_width} ${ax12_depth} ${ax12_height}"/>
+    </xacro:property>
     <xacro:property name="left_sho_pitch_block_origin">
         <origin xyz="0 0.45 0.14" rpy="0 0 0"/>
@@ -112,5 +117,5 @@
     </xacro:property>
     <xacro:property name="head_tilt_block_origin">
-        <origin xyz="-0.12 0 0.22" rpy="0 0 0"/>
+        <origin xyz="-0.12 0 0.222" rpy="0 0 0"/>
     </xacro:property>
     <xacro:property name="ax12_block_inertia">
@@ -166,5 +171,5 @@
             <xacro:insert_block name="torso_origin"/>
             <geometry>
-                <mesh filename="package://test_description/meshes2/torso.dae"/>
+                <mesh filename="package://${package_name}/${mesh_dir}/torso.dae"/>
             </geometry>
             <material name="orange"/>
@@ -193,5 +198,5 @@
             <xacro:insert_block name="left_sho_pitch_block_origin"/>
             <geometry>
-                <mesh filename="package://test_description/meshes2/left_sho_pitch.dae"/>
+                <mesh filename="package://${package_name}/${mesh_dir}/left_sho_pitch.dae"/>
             </geometry>
             <material name="black"/>
@@ -221,5 +226,5 @@
             <xacro:insert_block name="left_sho_pitch_bracket_origin"/>
             <geometry>
-                <mesh filename="package://test_description/meshes2/left_sho_pitch_bracket.dae"/>
+                <mesh filename="package://${package_name}/${mesh_dir}/left_sho_pitch_bracket.dae"/>
             </geometry>
             <material name="black"/>
@@ -249,5 +254,5 @@
             <xacro:insert_block name="left_sho_roll_block_origin"/>
             <geometry>
-                <mesh filename="package://test_description/meshes2/left_sho_roll.dae"/>
+                <mesh filename="package://${package_name}/${mesh_dir}/left_sho_roll.dae"/>
             </geometry>
             <material name="black"/>
@@ -275,5 +280,5 @@
             <xacro:insert_block name="left_elbow_bracket_origin"/>
             <geometry>
-                <mesh filename="package://test_description/meshes2/left_elbow_bracket.dae"/>
+                <mesh filename="package://${package_name}/${mesh_dir}/left_elbow_bracket.dae"/>
             </geometry>
             <material name="black"/>
@@ -302,5 +307,5 @@
             <xacro:insert_block name="left_elbow_block_origin"/>
             <geometry>
-                <mesh filename="package://test_description/meshes2/left_elbow_pitch.dae"/>
+                <mesh filename="package://${package_name}/${mesh_dir}/left_elbow_pitch.dae"/>
             </geometry>
             <material name="black"/>
@@ -327,5 +332,5 @@
             <xacro:insert_block name="left_hand_origin"/>
             <geometry>
-                <mesh filename="package://test_description/meshes2/left_hand.dae"/>
+                <mesh filename="package://${package_name}/${mesh_dir}/left_hand.dae"/>
             </geometry>
             <material name="black"/>
@@ -354,5 +359,5 @@
             <xacro:insert_block name="right_sho_pitch_block_origin"/>
             <geometry>
-                <mesh filename="package://test_description/meshes2/right_sho_pitch.dae"/>
+                <mesh filename="package://${package_name}/${mesh_dir}/right_sho_pitch.dae"/>
             </geometry>
             <material name="black"/>
@@ -382,5 +387,5 @@
             <xacro:insert_block name="right_sho_roll_block_origin"/>
             <geometry>
-                <mesh filename="package://test_description/meshes2/right_sho_roll.dae"/>
+                <mesh filename="package://${package_name}/${mesh_dir}/right_sho_roll.dae"/>
             </geometry>
             <material name="black"/>
@@ -408,5 +413,5 @@
             <xacro:insert_block name="right_elbow_bracket_origin"/>
             <geometry>
-                <mesh filename="package://test_description/meshes2/right_elbow_bracket.dae"/>
+                <mesh filename="package://${package_name}/${mesh_dir}/right_elbow_bracket.dae"/>
             </geometry>
             <material name="black"/>
@@ -437,5 +442,5 @@
             <xacro:insert_block name="right_sho_pitch_bracket_origin"/>
             <geometry>
-                <mesh filename="package://test_description/meshes2/right_sho_pitch_bracket.dae"/>
+                <mesh filename="package://${package_name}/${mesh_dir}/right_sho_pitch_bracket.dae"/>
             </geometry>
             <material name="black"/>
@@ -484,5 +489,5 @@
             <xacro:insert_block name="right_elbow_block_origin"/>
             <geometry>
-                <mesh filename="package://test_description/meshes2/right_elbow_pitch_fn.dae"/>
+                <mesh filename="package://${package_name}/${mesh_dir}/right_elbow_pitch_fn.dae"/>
             </geometry>
             <material name="black"/>
@@ -509,5 +514,5 @@
             <xacro:insert_block name="right_hand_origin"/>
             <geometry>
-                <mesh filename="package://test_description/meshes2/right_hand2.dae"/>
+                <mesh filename="package://${package_name}/${mesh_dir}/right_hand2.dae"/>
             </geometry>
             <material name="black"/>
@@ -529,13 +534,14 @@
     <link name="neck_pan_block">
         <collision>
+            <!-- <xacro:insert_block name="neck_pan_block_origin"/> -->
+            <origin xyz="-0.1385 0 0.218" rpy="1.5708 0 1.5708"/>
+            <geometry>
+                <xacro:insert_block name="ax12_block"/>
+            </geometry>
+        </collision>
+        <visual>
             <xacro:insert_block name="neck_pan_block_origin"/>
             <geometry>
-                <xacro:insert_block name="ax12_block"/>
-            </geometry>
-        </collision>
-        <visual>
-            <xacro:insert_block name="neck_pan_block_origin"/>
-            <geometry>
-                <mesh filename="package://test_description/meshes2/neck_base.dae"/>
+                <mesh filename="package://${package_name}/${mesh_dir}/neck_base.dae"/>
             </geometry>
             <material name="black"/>
@@ -554,13 +560,15 @@
     <link name="neck_pan_top_bracket">
         <collision>
+            <!-- <xacro:insert_block name="neck_pan_top_bracket_origin"/> -->
+            <origin xyz="0 0 0.0168" rpy="0 0 0" />
+            <geometry>
+                <!-- <xacro:insert_block name="ax12_block"/> -->
+                <box size="${ax12_height} ${ax12_depth} 0.058" />
+            </geometry>
+        </collision>
+        <visual>
             <xacro:insert_block name="neck_pan_top_bracket_origin"/>
             <geometry>
-                <xacro:insert_block name="ax12_block"/>
-            </geometry>
-        </collision>
-        <visual>
-            <xacro:insert_block name="neck_pan_top_bracket_origin"/>
-            <geometry>
-                <mesh filename="package://test_description/meshes2/neck_bottom.dae"/>
+                <mesh filename="package://${package_name}/${mesh_dir}/neck_bottom.dae"/>
             </geometry>
             <material name="black"/>
@@ -581,13 +589,15 @@
     <link name="neck_tilt_bottom_bracket">
         <collision>
+            <!-- <xacro:insert_block name="neck_tilt_bottom_bracket_origin"/> -->
+            <origin xyz="-0.12 0 0.07" rpy="0 0 0" />
+            <geometry>
+                <!-- <xacro:insert_block name="ax12_block"/> -->
+                <box size="${ax12_height} ${ax12_depth} 0.05" />
+            </geometry>
+        </collision>
+        <visual>
             <xacro:insert_block name="neck_tilt_bottom_bracket_origin"/>
             <geometry>
-                <xacro:insert_block name="ax12_block"/>
-            </geometry>
-        </collision>
-        <visual>
-            <xacro:insert_block name="neck_tilt_bottom_bracket_origin"/>
-            <geometry>
-                <mesh filename="package://test_description/meshes2/neck_top.dae"/>
+                <mesh filename="package://${package_name}/${mesh_dir}/head_top_bracket.dae"/>
             </geometry>
             <material name="black"/>
@@ -606,13 +616,14 @@
     <link name="head_tilt_block">
         <collision>
+            <!-- <xacro:insert_block name="head_tilt_block_origin"/> -->
+            <origin xyz="-0.12 0 0.222" rpy="1.5708 1.5708 1.5708"/>
+            <geometry>
+                <xacro:insert_block name="ax12_block"/>
+            </geometry>
+        </collision>
+        <visual>
             <xacro:insert_block name="head_tilt_block_origin"/>
             <geometry>
-                <xacro:insert_block name="ax12_block"/>
-            </geometry>
-        </collision>
-        <visual>
-            <xacro:insert_block name="head_tilt_block_origin"/>
-            <geometry>
-                <mesh filename="package://test_description/meshes2/head_tilt.dae"/>
+                <mesh filename="package://${package_name}/${mesh_dir}/head_tilt.dae"/>
             </geometry>
             <material name="black"/>

Commit message: Set torso collision

File: urdf/jimmy2.urdf.xacro (robot description, xacro)
@@ -163,7 +163,9 @@
     <link name="torso">
         <collision>
-            <xacro:insert_block name="torso_origin"/>
-            <geometry>
-                <xacro:insert_block name="ax12_block"/>
+            <!-- <xacro:insert_block name="torso_origin"/> -->
+            <origin xyz="0.13 0 -0.3" rpy="0 0 0" />
+            <geometry>
+                <!-- <xacro:insert_block name="ax12_block"/> -->
+                <box size="0.77 1.2 2.4"/>
             </geometry>
         </collision>

Commit message: Complete collision geometries

File: urdf/jimmy2.urdf.xacro (robot description, xacro)
@@ -38,4 +38,7 @@
         <origin xyz="0 0.45 0.14" rpy="0 0 0"/>
     </xacro:property>
+    <xacro:property name="left_sho_pitch_block_collision_origin">
+        <origin xyz="0 0.46 0.14" rpy="0 1.5708 0"/>
+    </xacro:property>
     <xacro:property name="left_sho_pitch_joint_origin">
         <origin xyz="0.14 0.655 0.14" rpy="0 0 0"/>
@@ -50,4 +53,7 @@
         <origin xyz="-0.01 0 -0.14" rpy="0 0 0"/>
     </xacro:property>
+    <xacro:property name="left_sho_roll_block_collision_origin">
+        <origin xyz="0 0 -0.14" rpy="0 0 1.5708"/>
+    </xacro:property>
     <xacro:property name="left_elbow_bracket_joint_origin">
         <origin xyz="0 0 -0.22" rpy="0 0 0"/>
@@ -65,7 +71,14 @@
         <origin xyz="0 0 -0.4" rpy="0 0 0"/>
     </xacro:property>
+    <xacro:property name="left_hand_collision_origin">
+        <origin xyz="0 0 -0.55" rpy="0 0 0"/>
+    </xacro:property>
+    <!-- Right Arm -->
     <xacro:property name="right_sho_pitch_block_origin">
         <origin xyz="0 -0.44 0.14" rpy="0 0 0"/>
     </xacro:property>
+    <xacro:property name="right_sho_pitch_block_collision_origin">
+        <origin xyz="0 -0.45 0.14" rpy="0 1.5708 0"/>
+    </xacro:property>
     <xacro:property name="right_sho_pitch_joint_origin">
         <origin xyz="0.14 -0.655 0.14" rpy="0 0 0"/>
@@ -80,4 +93,7 @@
         <origin xyz="-0.01 0 -0.14" rpy="0 0 0"/>
     </xacro:property>
+    <xacro:property name="right_sho_roll_block_collision_origin">
+        <origin xyz="0 0 -0.14" rpy="0 0 1.5708"/>
+    </xacro:property>
     <xacro:property name="right_elbow_bracket_joint_origin">
         <origin xyz="0 0 -0.22" rpy="0 0 0"/>
@@ -95,4 +111,8 @@
         <origin xyz="0 0 -0.4" rpy="0 0 0"/>
     </xacro:property>
+    <xacro:property name="right_hand_collision_origin">
+        <origin xyz="0 0 -0.55" rpy="0 0 0"/>
+    </xacro:property>
+    <!-- Neck/Head -->
     <xacro:property name="neck_pan_joint_origin">
         <origin xyz="0.2 0 0.87" rpy="0 0 0"/>
@@ -118,4 +138,7 @@
     <xacro:property name="head_tilt_block_origin">
         <origin xyz="-0.12 0 0.222" rpy="0 0 0"/>
+    </xacro:property>
+    <xacro:property name="bracket_collision_block">
+        <box size="0.0001 0.0001 0.0001"/>
     </xacro:property>
     <xacro:property name="ax12_block_inertia">
@@ -192,5 +215,5 @@
     <link name="left_sho_pitch_block">
         <collision>
-            <xacro:insert_block name="left_sho_pitch_block_origin"/>
+            <xacro:insert_block name="left_sho_pitch_block_collision_origin"/>
             <geometry>
                 <xacro:insert_block name="ax12_block"/>
@@ -222,5 +245,5 @@
             <xacro:insert_block name="left_sho_pitch_bracket_origin"/>
             <geometry>
-                <xacro:insert_block name="ax12_block"/>
+                <xacro:insert_block name="bracket_collision_block"/>
             </geometry>
         </collision>
@@ -248,5 +271,5 @@
     <link name="left_sho_roll_block">
         <collision>
-            <xacro:insert_block name="left_sho_roll_block_origin"/>
+            <xacro:insert_block name="left_sho_roll_block_collision_origin"/>
             <geometry>
                 <xacro:insert_block name="ax12_block"/>
@@ -276,5 +299,5 @@
             <xacro:insert_block name="left_elbow_bracket_origin"/>
             <geometry>
-                <xacro:insert_block name="ax12_block"/>
+                <xacro:insert_block name="bracket_collision_block"/>
             </geometry>
         </collision>
@@ -326,7 +349,8 @@
     <link name="left_hand">
         <collision>
-            <xacro:insert_block name="left_hand_origin"/>
-            <geometry>
-                <xacro:insert_block name="ax12_block"/>
+            <xacro:insert_block name="left_hand_collision_origin"/>
+            <geometry>
+                <!-- <xacro:insert_block name="ax12_block"/> -->
+                <box size="0.4 0.4 0.95" />
             </geometry>
         </collision>
@@ -353,19 +377,47 @@
     <link name="right_sho_pitch_block">
         <collision>
+            <xacro:insert_block name="right_sho_pitch_block_collision_origin"/>
+            <geometry>
+                <xacro:insert_block name="ax12_block"/>
+            </geometry>
+        </collision>
+        <visual>
             <xacro:insert_block name="right_sho_pitch_block_origin"/>
             <geometry>
-                <xacro:insert_block name="ax12_block"/>
-            </geometry>
-        </collision>
-        <visual>
+                <mesh filename="package://${package_name}/${mesh_dir}/right_sho_pitch.dae"/>
+            </geometry>
+            <material name="black"/>
+        </visual>
+        <inertial>
             <xacro:insert_block name="right_sho_pitch_block_origin"/>
-            <geometry>
-                <mesh filename="package://${package_name}/${mesh_dir}/right_sho_pitch.dae"/>
-            </geometry>
-            <material name="black"/>
-        </visual>
-        <inertial>
-            <xacro:insert_block name="right_sho_pitch_block_origin"/>
-            <mass value="${mass}"/>
+            <mass value="${mass}"/>
+            <xacro:insert_block name="ax12_block_inertia"/>
+        </inertial>
+    </link>
+    <joint name="right_sho_pitch" type="continuous">
+        <parent link="right_sho_pitch_block"/>
+        <child link="right_sho_pitch_bracket"/>
+        <origin xyz="0.14 -0.65 0.14" rpy="0 0 0"/>
+        <axis xyz="0 1 0"/>
+        <dynamics damping="0.7"/>
+    </joint>
+    <!-- right shoulder bracket -->
+    <link name="right_sho_pitch_bracket">
+        <collision>
+            <xacro:insert_block name="right_sho_pitch_bracket_origin"/>
+            <geometry>
+                <xacro:insert_block name="bracket_collision_block"/>
+            </geometry>
+        </collision>
+        <visual>
+            <xacro:insert_block name="right_sho_pitch_bracket_origin"/>
+            <geometry>
+                <mesh filename="package://${package_name}/${mesh_dir}/right_sho_pitch_bracket.dae"/>
+            </geometry>
+            <material name="black"/>
+        </visual>
+        <inertial>
+            <xacro:insert_block name="right_sho_pitch_bracket_origin"/>
+            <mass value="${bracket_mass}"/>
             <xacro:insert_block name="ax12_block_inertia"/>
         </inertial>
@@ -381,5 +433,5 @@
     <link name="right_sho_roll_block">
         <collision>
-            <xacro:insert_block name="right_sho_roll_block_origin"/>
+            <xacro:insert_block name="right_sho_roll_block_collision_origin"/>
             <geometry>
                 <xacro:insert_block name="ax12_block"/>
@@ -409,5 +461,5 @@
             <xacro:insert_block name="right_elbow_bracket_origin"/>
             <geometry>
-                <xacro:insert_block name="ax12_block"/>
+                <xacro:insert_block name="bracket_collision_block"/>
             </geometry>
         </collision>
@@ -426,52 +478,4 @@
     </link>
     <!-- end of Base Link -->
-    <joint name="right_sho_pitch" type="continuous">
-        <parent link="right_sho_pitch_block"/>
-        <child link="right_sho_pitch_bracket"/>
-        <origin xyz="0.14 -0.65 0.14" rpy="0 0 0"/>
-        <axis xyz="0 1 0"/>
-        <dynamics damping="0.7"/>
-    </joint>
-    <!-- right shoulder bracket -->
-    <link name="right_sho_pitch_bracket">
-        <collision>
-            <xacro:insert_block name="right_sho_pitch_bracket_origin"/>
-            <geometry>
-                <xacro:insert_block name="ax12_block"/>
-            </geometry>
-        </collision>
-        <visual>
-            <xacro:insert_block name="right_sho_pitch_bracket_origin"/>
-            <geometry>
-                <mesh filename="package://${package_name}/${mesh_dir}/right_sho_pitch_bracket.dae"/>
-            </geometry>
-            <material name="black"/>
-        </visual>
-        <inertial>
-            <xacro:insert_block name="right_sho_pitch_bracket_origin"/>
-            <mass value="${bracket_mass}"/>
-            <xacro:insert_block name="ax12_block_inertia"/>
-        </inertial>
-    </link>
-    <!-- <link name="right_elbow_block">
-        <collision>
-            <origin xyz="0 0 0" rpy="0 0 0"/>
-            <geometry>
-                <xacro:insert_block name="ax12_block"/>
-            </geometry>
-        </collision>
-        <visual>
-            <origin xyz="0 0 0" rpy="0 0 0"/>
-            <geometry>
-                <mesh filename="package://test_description/meshes/r_forearm2.dae"/>
-            </geometry>
-            <material name="black"/>
-        </visual>
-        <inertial>
-            <origin xyz="0 0 0" rpy="0 0 0"/>
-            <mass value="${mass}"/>
-            <xacro:insert_block name="ax12_block_inertia"/>
-        </inertial>
-    </link> -->
     <joint name="right_elbow_joint" type="continuous">
         <parent link="right_elbow_bracket"/>
@@ -508,7 +512,8 @@
     <link name="right_hand">
         <collision>
-            <xacro:insert_block name="right_hand_origin"/>
-            <geometry>
-                <xacro:insert_block name="ax12_block"/>
+            <xacro:insert_block name="right_hand_collision_origin"/>
+            <geometry>
+                <!-- <xacro:insert_block name="ax12_block"/> -->
+                <box size="0.4 0.4 0.95" />
             </geometry>
         </collision>

Commit message: Neck to revolute joint and self_collide

File: urdf/jimmy2.urdf.xacro (robot description, xacro)
@@ -532,5 +532,5 @@
     </link>
     <!-- end of Top Link -->
-    <joint name="neck_pan" type="continuous">
+    <joint name="neck_pan" type="revolute">
         <parent link="torso"/>
         <child link="neck_pan_block"/>
@@ -538,4 +538,5 @@
         <axis xyz="0 0 1"/>
         <dynamics damping="0.7"/>
+        <limit lower="-1.6807" upper="1.6807" effort="0.5" velocity="0.7"/>
     </joint>
     <link name="neck_pan_block">
@@ -587,5 +588,5 @@
         </inertial>
     </link>
-    <joint name="neck_tilt_bottom_bracket_passive_joint" type="continuous">
+    <joint name="neck_tilt_bottom_bracket_joint" type="revolute">
         <parent link="neck_pan_top_bracket" />
         <child link="neck_tilt_bottom_bracket" />
@@ -593,4 +594,5 @@
         <axis xyz="0 1.0 0"/>
         <dynamics damping="0.7"/>
+        <limit lower="-0.2807" upper="0.5807" effort="0.5" velocity="0.7"/>
     </joint>
     <link name="neck_tilt_bottom_bracket">
